File: MM Design/MM Power Subsystem.kicad_pcb (KiCad board)
At the start: 2 copper layers, 80 x 79 mm, 110 parts, among them J2 Conn_02x16_Odd_Even, J3 Conn_01x02_Pin, J4 USB_C_Receptacle_USB2.0_16P, SW1 SW_SPDT, U10 LMR33630ADDA, U11 CH224K, U12 TPS22929D, U13 TPS22929D, U14 LMR33630ADDA, U15 INA219BIDCNR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

Commit message: Add files via upload
Connections:
- SW1 pad 1: Battery -> BATT
- TP20 pad 1: Battery -> BATT
Routing:
- net BATT: track 178.9 -> 191.5 mm
- net Battery: track 12.6 -> 0.00 mm
