File: MM Design/MM Power Subsystem.kicad_sch (KiCad schematic)
At the start: 79 parts, among them J2 Conn_02x16_Odd_Even, J3 Conn_01x02_Pin, J4 USB_C_Receptacle_USB2.0_16P, SW1 SW_SPDT, U11 CH224K, U12 TPS22929D, U13 TPS22929D, U15 INA219BIDCNR, U4 MIC5219YMM, U5 TPS613222ADBV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

Commit message: Add files via upload
Parts:
- removed C20: 10uF, Capacitor_SMD:C_0402_1005Metric_Pad0.74x0.62mm_HandSolder, symbol Device:C_Small
- removed R2: 150k, Resistor_SMD:R_0402_1005Metric_Pad0.72x0.64mm_HandSolder, symbol Device:R_Small_US
- removed R29: 3m, Resistor_SMD:R_Shunt_Ohmite_LVK20, symbol Device:R_Shunt_US
- removed R3: 100k, Resistor_SMD:R_0402_1005Metric_Pad0.72x0.64mm_HandSolder, symbol Device:R_Small_US
- removed SW1: SW_SPDT, Button_Switch_THT:SW_Slide_SPDT_Angled_CK_OS102011MA1Q, symbol Switch:SW_SPDT
- removed U4: MIC5219YMM, Package_SO:MSOP-8_3x3mm_P0.65mm, symbol Regulator_Linear:MIC5219YMM
- added C8: 1uF, Capacitor_SMD:C_0402_1005Metric_Pad0.74x0.62mm_HandSolder, symbol Device:C
- added R1: 3m, symbol Device:R_Shunt_US
- added S1: Tactile Button, 160gf, PCM_JLCPCB:SW-SMD_4P-L5.1-W5.1-P3.70-LS6.5-TL-2, symbol PCM_JLCPCB-Connectors_Buttons:Tactile Button, 160gf
- added U1: AP2112K-3.3, Package_TO_SOT_SMD:SOT-23-5, symbol Regulator_Linear:AP2112K-3.3
Connections:
- net 3V3 Out: now also U1.5 (VOUT)
- net 5V Out: now also C8.1, U1.1 (VIN), U1.3 (EN)
- net Batt: now also R1.1
- net Battery: now also S1.4 (D)
- net GND: now also C8.2, U1.2 (GND)
- net at U15.1 (VIN+): now also R1.2
- net at U15.2 (VIN-): now also R1.3
- new net: R1.4, S1.1 (A)
Other:
- moved on the sheet: TP20
